File: PCB/Rosa.kicad_pcb (KiCad board)
At the start: 2 copper layers, 33.7 x 40.4 mm, 16 parts

Commit message: Add files via upload
Other:
- board text added: "Thanks also to Kavanoz, sparxUK, call286, KarlosJackel, erikbakke, Vincent Price, Dr. Chris, RRG, ElectronAsh, Neodeus, Houston, RetroGameRevival, pa1mer, TRU, Cathers, mafitzee, Andy T, Wrangler, Pillock, Tom Meades, Brian Gerfort, Hey Birt!, Andrew Littleboy, StuRoRo, CRG, Retro Krazy, gravitone, Chucky, Game Tech Refuge, SLR, Plan C, bitmapbureau, thegirlg33k, Four X, and Stefan Skotte for say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"
- board text removed: "Thanks also to Kavanoz, sparxUK, call286, KarlosJackel, erikbakke, Vincent Price, Dr. Chris, ElectronAsh, Neodeus, Houston, RetroGameRevival, pa1mer, TRU, Cathers, mafitzee, Andy T, Wrangler, Pillock, Tom Meades, Andrew Littleboy, StuRoRo, CRG, Retro Krazy, gravitone, Four X, Game Tech Refuge, SLR, Plan C, bitmapbureau, thegirlg33k, and Stefan Skotte for saying {dblquote}Is it ready yet????{dblqu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"
Changed lines of the file:
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@@
     (effects (font (size 1 1) (thickness 0.15)) (justify left bottom mirror))
   )
-  (gr_text "Thanks also to Kavanoz, sparxUK, \ncall286, KarlosJackel, erikbakke,\nVincent Price, Dr. Chris, \nElectronAsh, Neodeus, Houston,\nRetroGameRevival, pa1mer, TRU,\nCathers,             mafitzee,\nAndy T,              Wrangler, \nPillock,             Tom Meades, \n \nAndrew Littleboy, StuRoRo, CRG, \nRetro Krazy, gravitone, Four X, \nGame Tech Refuge, SLR, Plan C,\nbitmapbureau, thegirlg33k, \n and Stefan Skotte for saying\n{dblquote}Is it ready yet????{dblquote}!  \n           Need more space..." (at 29.1592 28.8544) (layer "B.SilkS")
+  (gr_text "Thanks also to Kavanoz, sparxUK, \ncall286, KarlosJackel, erikbakke,\nVincent Price, Dr. Chris, RRG,\nElectronAsh, Neodeus, Houston,\nRetroGameRevival, pa1mer, TRU,\nCathers,             mafitzee,\nAndy T,              Wrangler, \nPillock,             Tom Meades, \nBrian Gerfort,	  Hey Birt!,\nAndrew Littleboy, StuRoRo, CRG, \nRetro Krazy, gravitone, Chucky,\nGame Tech Refuge, SLR, Plan C,\nbitmapbureau, thegirlg33k, Four X, \n and Stefan Skotte for saying\n{dblquote}Is it ready yet????{dblquote}!  \n           Need more space..." (at 29.1592 28.8544) (layer "B.SilkS")
     (effects (font (size 0.7 0.7) (thickness 0.15)) (justify left bottom mirror))
   )

Commit message: Add files via upload
Parts:
- C3, C4: renamed from  
Other:
- board text added: "RC2a"
- board text removed: "RC2"

Commit message: Update Rosa.kicad_pcb
Additional credit.
Other:
- board text added: "RC2b"
- board text added: "Thanks also to Kavanoz, sparxUK, call286, KarlosJackel, erikbakke, Vincent Price, Dr. Chris, RRG, ElectronAsh, Neodeus, Houston, RetroGameRevival, pa1mer, TRU, Cathers, mafitzee, Andy T, Wrangler, Pillock, Tom Meades, Brian Gerfort, Hey Birt!, Andrew Littleboy, StuRoRo, CRG, Retro Krazy, gravitone, Chucky, Game Tech Refuge, SLR, Plan C, bitmapbureau, thegirlg33k, Four X, Zarchos, and Stefan Skott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"
- board text removed: "RC2a"
- board text removed: "Thanks also to Kavanoz, sparxUK, call286, KarlosJackel, erikbakke, Vincent Price, Dr. Chris, RRG, ElectronAsh, Neodeus, Houston, RetroGameRevival, pa1mer, TRU, Cathers, mafitzee, Andy T, Wrangler, Pillock, Tom Meades, Brian Gerfort, Hey Birt!, Andrew Littleboy, StuRoRo, CRG, Retro Krazy, gravitone, Chucky, Game Tech Refuge, SLR, Plan C, bitmapbureau, thegirlg33k, Four X, and Stefan Skotte for say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"
